File: pcb_layout_phaser90/pcb_layout_phaser90.kicad_pcb (KiCad board)
At the start: 2 copper layers, 0 parts

Commit message: changes to PCB-desing
Parts:
- added C1: 10n, Capacitor_THT:C_Disc_D3.0mm_W1.6mm_P2.50mm, F.Cu at (114.0, 82.6)
- added C10: 47µ, Capacitor_THT:CP_Radial_D8.0mm_P5.00mm, F.Cu at (120.5, 95.4)
- added C11: 10n, Capacitor_THT:C_Disc_D3.0mm_W1.6mm_P2.50mm, F.Cu at (114.0, 101.5)
- added C2: 47n, Capacitor_THT:C_Disc_D3.0mm_W1.6mm_P2.50mm, F.Cu at (114.0, 85.8)
- added C3: 47n, Capacitor_THT:C_Disc_D3.0mm_W1.6mm_P2.50mm, F.Cu at (49.7, 135.7)
- added C4: 47n, Capacitor_THT:C_Disc_D3.0mm_W1.6mm_P2.50mm, F.Cu at (61.4, 139.1)
- added C5: 47n, Capacitor_THT:C_Disc_D3.0mm_W1.6mm_P2.50mm, F.Cu at (114.0, 88.9)
- added C6: 47n, Capacitor_THT:C_Disc_D3.0mm_W1.6mm_P2.50mm, F.Cu at (114.0, 92.1)
- added C7: 10n, Capacitor_THT:C_Disc_D3.0mm_W1.6mm_P2.50mm, F.Cu at (114.0, 95.2)
- added C8: 10µ, Capacitor_THT:CP_Radial_D8.0mm_P5.00mm, F.Cu at (120.5, 85.8)
- added C9: 47n, Capacitor_THT:C_Disc_D3.0mm_W1.6mm_P2.50mm, F.Cu at (114.0, 98.4)
- added D1: LED, LED_THT:LED_D3.0mm_Clear, F.Cu at (129.5, 99.1)
- added D2: 1N4733A, Diode_THT:D_DO-41_SOD81_P10.16mm_Horizontal, F.Cu at (129.7, 83.2)
- added Q1: BF265B, Package_TO_SOT_THT:TO-92_Inline, F.Cu at (114.4, 37.8)
- added Q2: BF265B, Package_TO_SOT_THT:TO-92_Inline, F.Cu at (114.4, 43.6)
- added Q3: BF265B, Package_TO_SOT_THT:TO-92_Inline, F.Cu at (114.4, 49.4)
- added Q4: BF265B, Package_TO_SOT_THT:TO-92_Inline, F.Cu at (114.4, 55.2)
- added Q5: 2N3906, Package_TO_SOT_THT:TO-92_Inline, F.Cu at (114.4, 61.0)
- added Q6: 2N3904, Package_TO_SOT_THT:TO-92_Inline, F.Cu at (114.4, 66.8)
- added R1: 2.2M, Resistor_THT:R_Axial_DIN0411_L9.9mm_D3.6mm_P12.70mm_Horizontal, F.Cu at (97.7, 37.2)
- added R10: 10k, Resistor_THT:R_Axial_DIN0411_L9.9mm_D3.6mm_P12.70mm_Horizontal, F.Cu at (97.7, 52.6)
- added R11: 22k, Resistor_THT:R_Axial_DIN0411_L9.9mm_D3.6mm_P12.70mm_Horizontal, F.Cu at (97.7, 57.8)
- added R12: 10k, Resistor_THT:R_Axial_DIN0411_L9.9mm_D3.6mm_P12.70mm_Horizontal, F.Cu at (97.7, 62.9)
- added R13: 10k, Resistor_THT:R_Axial_DIN0411_L9.9mm_D3.6mm_P12.70mm_Horizontal, F.Cu at (97.7, 68.1)
- added R14: 22k, Resistor_THT:R_Axial_DIN0411_L9.9mm_D3.6mm_P12.70mm_Horizontal, F.Cu at (36.5, 35.2)
- added R15: 10k, Resistor_THT:R_Axial_DIN0411_L9.9mm_D3.6mm_P12.70mm_Horizontal, F.Cu at (36.5, 40.4)
- added R16: 150k, Resistor_THT:R_Axial_DIN0411_L9.9mm_D3.6mm_P12.70mm_Horizontal, F.Cu at (97.7, 73.2)
- added R17: 150k, Resistor_THT:R_Axial_DIN0411_L9.9mm_D3.6mm_P12.70mm_Horizontal, F.Cu at (97.7, 78.4)
- added R18: 150k, Resistor_THT:R_Axial_DIN0411_L9.9mm_D3.6mm_P12.70mm_Horizontal, F.Cu at (97.7, 83.5)
- added R19: 47k, Resistor_THT:R_Axial_DIN0411_L9.9mm_D3.6mm_P12.70mm_Horizontal, F.Cu at (36.5, 61.0)
- added R2: 10k, Resistor_THT:R_Axial_DIN0411_L9.9mm_D3.6mm_P12.70mm_Horizontal, F.Cu at (97.7, 42.3)
- added R20: 150k, Resistor_THT:R_Axial_DIN0411_L9.9mm_D3.6mm_P12.70mm_Horizontal, F.Cu at (36.5, 66.1)
- added R21: 150k, Resistor_THT:R_Axial_DIN0411_L9.9mm_D3.6mm_P12.70mm_Horizontal, F.Cu at (97.7, 88.7)
- added R22: 2k, Resistor_THT:R_Axial_DIN0411_L9.9mm_D3.6mm_P12.70mm_Horizontal, F.Cu at (97.7, 93.8)
- added R23: 470k, Resistor_THT:R_Axial_DIN0411_L9.9mm_D3.6mm_P12.70mm_Horizontal, F.Cu at (97.7, 99.0)
- added R24: 150k, Resistor_THT:R_Axial_DIN0411_L9.9mm_D3.6mm_P12.70mm_Horizontal, F.Cu at (97.7, 104.1)
- added R25: 10k, Resistor_THT:R_Axial_DIN0411_L9.9mm_D3.6mm_P12.70mm_Horizontal, F.Cu at (97.7, 109.3)
- added R26: 500, Resistor_THT:R_Axial_DIN0411_L9.9mm_D3.6mm_P12.70mm_Horizontal, F.Cu at (97.7, 114.4)
- added R27: 4.7M, Resistor_THT:R_Axial_DIN0411_L9.9mm_D3.6mm_P12.70mm_Horizontal, F.Cu at (97.7, 119.6)
- added R28: 1M, Resistor_THT:R_Axial_DIN0411_L9.9mm_D3.6mm_P12.70mm_Horizontal, F.Cu at (97.7, 124.7)
- added R29: 10k, Resistor_THT:R_Axial_DIN0411_L9.9mm_D3.6mm_P12.70mm_Horizontal, F.Cu at (97.7, 129.9)
- added R3: 2.2M, Resistor_THT:R_Axial_DIN0411_L9.9mm_D3.6mm_P12.70mm_Horizontal, F.Cu at (97.7, 47.5)
- added R4: 10k, Resistor_THT:R_Axial_DIN0411_L9.9mm_D3.6mm_P12.70mm_Horizontal, F.Cu at (19.9, 35.2)
- added R5: 10k, Resistor_THT:R_Axial_DIN0411_L9.9mm_D3.6mm_P12.70mm_Horizontal, F.Cu at (19.9, 40.4)
- added R6: 22k, Resistor_THT:R_Axial_DIN0411_L9.9mm_D3.6mm_P12.70mm_Horizontal, F.Cu at (19.9, 45.5)
- added R7: 10k, Resistor_THT:R_Axial_DIN0411_L9.9mm_D3.6mm_P12.70mm_Horizontal, F.Cu at (19.9, 50.7)
- added R8: 22k, Resistor_THT:R_Axial_DIN0411_L9.9mm_D3.6mm_P12.70mm_Horizontal, F.Cu at (19.9, 55.8)
- added R9: 10k, Resistor_THT:R_Axial_DIN0411_L9.9mm_D3.6mm_P12.70mm_Horizontal, F.Cu at (19.9, 61.0)
- added RV1: 470k, Potentiometer_THT:Potentiometer_Alps_RK163_Single_Horizontal, F.Cu at (205.2, 42.9)
- added RV2: 100k, Potentiometer_THT:Potentiometer_Bourns_3386F_Vertical, F.Cu at (130.7, 93.4)
- added RV3: 250k, Potentiometer_THT:Potentiometer_Alps_RK163_Single_Horizontal, F.Cu at (231.1, 42.8)
- added U1: TL072, Package_DIP:DIP-8_W7.62mm, F.Cu at (114.0, 71.4)
- added U2: TL072, Package_DIP:DIP-8_W7.62mm, F.Cu at (124.8, 71.4)
- added U3: TL072, Package_DIP:DIP-8_W7.62mm, F.Cu at (135.6, 71.4)
Routing:
- net Mixer_output: track 0.00 -> 5.00 mm
Other:
- board text added: "-CHECK TL072 POWER RAILS"
